File: DigitalDash/DriverPanel.brd (EAGLE design)
At the start: 216.8 x 87.5 mm, 108 parts, among them IC1 7805T, J2 DT15-4P, J3 DT15-4P, U1 IS31FL3741_QFN60, U2 IS31FL3741_QFN60

Commit message: stuff
Parts:
- added R83, R84, R85, R86: 10k, rcl:R0805
Connections:
- removed net VCC: C1.1, C10.1, C11.1, C12.1, C2.1, C3.1, C4.1, C6.1, C7.1, C8.1, J1.4, U1.14, U1.15, U1.25, U2.14, U2.15, U2.25
- new net BUTTON1: R84.2, S1.3, U$5.6
- new net BUTTON2: R83.2, S2.3, U$5.5
- new net BUTTON3: R86.2, S3.3, U$5.9
- new net BUTTON4: R85.2, S4.3, U$5.10
- net 3V3: now also S1.1, S2.1, S3.1, S4.1
- net 5VDC: now also C1.1, C10.1, C11.1, C12.1, C2.1, C3.1, C4.1, C6.1, C7.1, C8.1, J1.4, U$5.USB, U1.14, U1.15, U1.25, U2.14, U2.15, U2.25
- net GND: now also R83.1, R84.1, R85.1, R86.1, U$5.GND, U$5.GND2
Routing:
- net BUTTON4: track 0.00 -> 147.0 mm, vias 0 -> 1
- net 3V3: track 226.3 -> 372.5 mm, vias 2 -> 4
- net BUTTON3: track 0.00 -> 137.8 mm, vias 0 -> 1
- net CANH: track 0.00 -> 124.1 mm
- net CANL: track 0.00 -> 117.2 mm
- net 5VDC: track 64.4 -> 155.5 mm, vias 0 -> 7
- net BUTTON1: track 0.00 -> 86.3 mm, vias 0 -> 1
- net BUTTON2: track 0.00 -> 84.4 mm, vias 0 -> 1
- net VCC: track 81.7 -> 0.00 mm, vias 5 -> 0
- net GND: track 153.6 -> 168.9 mm, vias 10 -> 12
- added copper zone on layer 16, net 5VDC
- removed copper zone on layer 16, net VCC
