File: DigitalDash/DriverPanel.sch (EAGLE design)
At the start: 108 parts, among them IC1 7805T, J2 DT15-4P, J3 DT15-4P, U1 IS31FL3741_QFN60, U2 IS31FL3741_QFN60

Commit message: stuff
Parts:
- added R83, R84, R85, R86: 10k, rcl:R-US_R0805
Connections:
- removed net VCC: C1.1, C10.1, C11.1, C12.1, C2.1, C3.1, C4.1, C6.1, C7.1, C8.1, J1.4, U1.AVCC, U1.PVCC1, U1.PVCC2, U2.AVCC, U2.PVCC1, U2.PVCC2
- new net BUTTON1: R84.2, S1.2, U$5.6
- new net BUTTON2: R83.2, S2.2, U$5.5
- new net BUTTON3: R86.2, S3.2, U$5.9
- new net BUTTON4: R85.2, S4.2, U$5.10
- net 3V3: now also S1.1, S2.1, S3.1, S4.1
- net 5VDC: now also C1.1, C10.1, C11.1, C12.1, C2.1, C3.1, C4.1, C6.1, C7.1, C8.1, J1.4, U$5.USB, U1.AVCC, U1.PVCC1, U1.PVCC2, U2.AVCC, U2.PVCC1, U2.PVCC2
- net GND: now also R83.1, R84.1, R85.1, R86.1, U$5.GND
Other:
- moved on the sheet: S1, S2, S3, S4
