File: DigitalDash/CANMosfetExtension.sch (EAGLE design)
At the start: 97 parts, among them IC1 7805T, J1 DT15-4P, J3 DT15-4P, Q10 IRFR9014TRPBF-BE3, Q11 IRFR9014TRPBF-BE3, Q12 IRFR9014TRPBF-BE3, Q13 IRFR9014TRPBF-BE3, Q14 IRFR9014TRPBF-BE3, Q15 IRFR9014TRPBF-BE3, Q16 IRFR9014TRPBF-BE3, Q9 IRFR9014TRPBF-BE3, U1 ATMEGA328P_TQFP, U10 LTV-817S, U11 LTV-817S, U2 MCP2515, U3 MCP2551, U4 LTV-817S, U5 LTV-817S, U6 LTV-817S, U7 LTV-817S, U8 LTV-817S, U9 LTV-817S, Y1 16MHz, Y2 8MHz

Commit message: update a lot
Parts:
- removed C1, C2, C3, C4: 22pF, SparkFun-Capacitors:22PF-0603-50V-5%
- removed C5: 1uF, SparkFun-Capacitors:22PF-0603-50V-5%
- removed D10, D11, D12, D13, D14, D15, D16: (no value), diode:DIODE-SOD123
- removed D8: (no value), SparkFun-LED:LED0603
- removed IC1: 7805T, linear:7805T
- removed J2: (no value), SparkFun-Connectors:CONN_03X2SHROUD
- removed J3: DT15-4P, DT15-4P:DT15-4P
- removed J7: (no value), SparkFun-Connectors:CONN_03LOCK
- removed Q10, Q11, Q12, Q13, Q14, Q15, Q16: IRFR9014TRPBF-BE3, SamacSys_Parts:IRFR9014TRPBF-BE3
- removed R26, R8: 3.3k, SparkFun-Resistors:1KOHM-0603-1/10W-1%
- removed R27: 33k, SparkFun-Resistors:1KOHM-0603-1/10W-1%
- removed R29, R30, R31, R32, R33, R34, R35: 1K, SparkFun-Resistors:1KOHM-0603-1/10W-1%
- removed R7: 470R, SparkFun-Resistors:1KOHM-0603-1/10W-1%
- removed U$1, U$2, U$3, U$4: KEYSTONEM3, KeystoneSMD:KEYSTONEM3
- removed U10, U11: LTV-817S, SamacSys_Parts:LTV-817S
- removed U3: MCP2551, SparkFun-IC-Comms:MCP2551
- removed X4: (no value), con-wago-500:W237-102
- removed Y1: 16MHz, SparkFun-Clocks:CRYSTAL-8MHZSMD-HC49UP
- removed Y2: 8MHz, SparkFun-Clocks:CRYSTAL-8MHZSMD-HC49UP
- added Q2, Q3, Q4: IRFR9014TRPBF-BE3, SamacSys_Parts:IRFR9014TRPBF-BE3
- added X1: (no value), con-wago-500:W237-102
- D3, D5, D7: device SparkFun-LED:LED0603 -> diode:DIODE-SOD123
- J1: value DT15-4P -> (none); device DT15-4P:DT15-4P -> SparkFun-Connectors:CONN_03LOCK
- R1: value 1k -> 470R
- R10, R16: value 470R -> 470
- R11: value 3.3k -> 4.7K
- R12: value 33k -> 470
- R13: value 470R -> 4.7K
- R14: value 3.3k -> 470
- R15, R9: value 33k -> 4.7K
- R17, R5: value 3.3k -> 470R
- R18, R6: value 33k -> 3.3k
- R19: value 470R -> 33k
- R2: value 10k -> 3.3k
- R20: value 3.3k -> 33k
- R21: value 33k -> 1K
- R25, R4: value 470R -> 1K
- R3: value 10k -> 33k
- U1: value ATMEGA328P_TQFP -> LTV-817S; device SparkFun-IC-Microcontroller:ATMEGA328P_TQFP -> SamacSys_Parts:LTV-817S
- U2: value MCP2515 -> LTV-817S; device SparkFun-IC-Comms:MCP2515(MCP2510)SO -> SamacSys_Parts:LTV-817S
Connections:
- removed net ARDUINO1: U1.PD1(TXD)
- removed net ARDUINO14: R13.1, R31.2, U1.PC0(ADC0)
- removed net ARDUINO15: R10.1, R30.2, U1.PC1(ADC1)
- removed net ARDUINO16: R29.2, R7.1, U1.PC2(ADC2)
- removed net ARDUINO17: R28.2, R4.1, U1.PC3(ADC3)
- removed net ARDUINO5: R25.1, R35.2, U1.PD5(T1)
- removed net ARDUINO6: R22.1, R34.2, U1.PD6(AIN0)
- removed net ARDUINOA6: R19.1, R33.2, U1.ADC6
- removed net ARDUINOA7: R16.1, R32.2, U1.ADC7
- removed net CANH: J1.2, J3.2, U3.CANH
- removed net CANL: J1.3, J3.3, U3.CANL
- removed net CAN_INT: U1.PD2(INT0), U2>NAME.INT
- removed net CS: U1.PB2(SS/OC1B), U2>NAME.CS
- removed net MISO: J2.1, U1.PB4(MISO), U2>NAME.SO
- removed net MOSI: J2.4, U1.PB3(MOSI/OC2), U2>NAME.SI
- removed net N$21: R16.2, U8.ANODE
- removed net N$22: R17.1, U8.COLLECTOR
- removed net N$23: D13.A, Q13.G, R17.2, R18.1
- removed net N$24: R19.2, U9.ANODE
- removed net N$25: R20.1, U9.COLLECTOR
- removed net N$26: D14.A, Q14.G, R20.2, R21.1
- removed net N$27: R22.2, U10.ANODE
- removed net N$28: R23.1, U10.COLLECTOR
- removed net N$29: D15.A, Q15.G, R23.2, R24.1
- removed net N$30: R25.2, U11.ANODE
- removed net N$31: R26.1, U11.COLLECTOR
- removed net N$32: D16.A, Q16.G, R26.2, R27.1
- removed net N$34: D2.A, R29.1
- removed net N$35: D3.A, R30.1
- removed net N$36: D4.A, R31.1
- removed net N$37: D5.A, R32.1
- removed net N$38: D6.A, R33.1
- removed net N$39: D7.A, R34.1
- removed net N$40: D8.A, R35.1
- removed net N$6: C3.2, U1.PB6(XTAL1/TOSC1), Y1.2
- removed net OUTPUT5: Q13.S, X6-1.KL
- removed net OUTPUT6: Q14.S, X7-1.KL
- removed net OUTPUT7: Q15.S, X8-1.KL
- removed net OUTPUT8: Q16.S, X9-1.KL
- removed net RST: J2.5, R1.2, U1.PC6(/RESET)
- removed net SCK: J2.3, U1.PB5(SCK), U2>NAME.SCK
- new net IN5: R10.2, X5-1.KL
- new net IN6: R12.2, X6-1.KL
- new net IN7: R14.2, X7-1.KL
- new net IN8: R16.2, X8-1.KL
- net +12VCC1: now also D3.C, D5.C, D7.C, J1.2, J1.3, Q2.D, Q3.D, Q4.D, R19.2, R20.2, R3.2; no longer D10.C, D11.C, D12.C, D13.C, D14.C, D15.C, D16.C, IC1.VI, J3.1, J6.1, J6.2, J6.3, Q10.D, Q11.D, Q12.D, Q13.D, Q14.D, Q15.D, Q16.D, R12.2, R15.2, R18.2, R21.2, R27.2, R6.2, R9.2
- net ARDUINO0: now also R21.2, R5.1; no longer U1.PD0(RXD)
- net ARDUINO18: now also R9.1, U4.COLLECTOR; no longer U1.PC4(ADC4/SDA)
- net ARDUINO19: now also R22.1, R25.2; no longer U1.PC5(ADC5/SCL)
- net ARDUINO3: now also R1.1, R4.2; no longer U1.PD3(INT1)
- net ARDUINO4: now also R17.1, R28.2; no longer U1.PD4(XCK/T0)
- net ARDUINO7: now also R15.1, U7.COLLECTOR; no longer U1.PD7(AIN1)
- net ARDUINO8: now also R13.1, U6.COLLECTOR; no longer U1.PB0(ICP)
- net ARDUINO9: now also R11.1, U5.COLLECTOR; no longer U1.PB1(OC1A)
- net GND: now also J6.1, J6.2, J6.3, U1.CATHODE, U1.EMITTER, U2.CATHODE, U2.EMITTER, X1-2.KL; no longer C1.1, C2.1, C3.1, C4.1, C5.1, D3.C, D5.C, D7.C, D8.C, IC1.GND, J1.4, J2.6, J3.4, J7.1, J7.2, J7.3, R2.2, U1.AGND, U1.AREF, U1.GND@3, U1.GND@5, U10.CATHODE, U10.EMITTER, U11.CATHODE, U11.EMITTER, U2P.VSS, U3.VSS, X4-2.KL, X5-2.KL, X6-2.KL, X7-2.KL, X8-2.KL
- net N$1: now also R18.1, U9.COLLECTOR; no longer U2>NAME.TXCAN, U3.TXD
- net N$10: now also R12.1, U5.ANODE; no longer R5.1, U4.COLLECTOR
- net N$11: now also R18.2, R19.1; no longer R5.2, R6.1
- net N$12: now also R14.1, U6.ANODE; no longer R7.2, U5.ANODE
- net N$13: now also R6.1, U2.COLLECTOR; no longer R8.1, U5.COLLECTOR
- net N$14: now also R16.1, U7.ANODE; no longer D10.A, Q10.G, R8.2, R9.1
- net N$15: now also D5.A, Q3.G, R20.1, R6.2; no longer R10.2, U6.ANODE
- net N$16: now also D4.A, R21.1; no longer R11.1, U6.COLLECTOR
- net N$17: now also R22.2, U8.ANODE; no longer D11.A, Q11.G, R11.2, R12.1
- net N$18: now also R23.1, U8.COLLECTOR; no longer R13.2, U7.ANODE
- net N$19: now also D7.A, Q4.G, R23.2, R24.1; no longer R14.1, U7.COLLECTOR
- net N$2: now also R1.2, U1.ANODE; no longer U2>NAME.RXCAN, U3.RXD
- net N$20: now also D6.A, R25.1; no longer D12.A, Q12.G, R14.2, R15.1
- net N$3: now also R2.1, U1.COLLECTOR; no longer C2.2, U2>NAME.OSC2, Y2.1
- net N$4: now also R5.2, U2.ANODE; no longer C1.2, U2>NAME.OSC1, Y2.2
- net N$5: now also D3.A, Q2.G, R2.2, R3.1; no longer C4.2, U1.PB7(XTAL2/TOSC2), Y1.1
- net N$7: now also D2.A, R4.1; no longer R2.1, U3.RS
- net N$8: now also R10.1, U4.ANODE; no longer R3.2, U2>NAME.RESET
- net N$9: now also R17.2, U9.ANODE; no longer R4.2, U4.ANODE
- net OUTPUT1: now also X9-1.KL; no longer X2-1.KL
- net OUTPUT2: now also Q2.S, X1-1.KL; no longer Q10.S, X3-1.KL
- net OUTPUT3: now also Q3.S, X2-1.KL; no longer Q11.S, X4-1.KL
- net OUTPUT4: now also Q4.S, X3-1.KL; no longer Q12.S, X5-1.KL
- net VCC: now also R11.2, R13.2, R15.2, R9.2; no longer C5.2, IC1.VO, J2.2, R1.1, R3.1, U1.AVCC, U1.VCC@4, U1.VCC@6, U2P.VDD, U3.VDD
Other:
- moved on the sheet: D1, D2, D4, D6, D9, J4, J5, J6, Q9, R1, R10, R11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
