File: DigitalDash/MOSFETboard.brd (EAGLE design)
At the start: 196.8 x 40.3 mm, 65 parts, among them IC1 7805T, J1 DT15-4P, J3 DT15-4P, J4 AVR_SPI_PROG_3X22X3_LOCK, U1 ATMEGA328P_TQFP, U10 LTV-817S, U11 LTV-817S, U2 MCP2515, U3 MCP2551, U4 LTV-817S, U5 LTV-817S, U6 LTV-817S, U7 LTV-817S, U8 LTV-817S, U9 LTV-817S, Y1 16MHz, Y2 8MHz

Commit message: update a lot
Parts:
- removed X1: (no value), con-wago-500:W237-102
- added C5: 1uF, SparkFun-Capacitors:0603
- added D1, D2, D3, D4, D5, D6, D7, D8: (no value), SparkFun-LED:LED-0603
- added D10, D11, D12, D13, D14, D15, D16, D9: (no value), diode:SOD123
- added J2: (no value), SparkFun-Connectors:2X3-SHROUDED
- added J5, J6, J7: (no value), SparkFun-Connectors:1X03_LOCK
- added R28, R29, R30, R31, R32, R33, R34, R35: 1K, SparkFun-Resistors:0603
- added U$1, U$2, U$3, U$4: KEYSTONEM3, KeystoneSMD:M3SMDSTANDOFF
- J4: value AVR_SPI_PROG_3X22X3_LOCK -> (none); device SparkFun-Connectors:2X3_LOCK -> SparkFun-Connectors:1X08_LOCK
- Q10, Q11, Q12, Q13, Q14, Q15, Q16, Q9: value (none) -> IRFR9014TRPBF-BE3
- moved J4 26.0 mm to (136.4, 2.16), turned to 0 degrees
- moved C3 14.2 mm to (152.7, 10.7)
- moved R1 14.0 mm to (123.7, 3.81)
- moved C4 10.7 mm to (144.0, 10.7), turned to 180 degrees
- moved R2 6.73 mm to (68.8, 1.27), turned to 0 degrees
- moved J3 5.46 mm to (12.7, 17.1)
- moved IC1 5.34 mm to (55.9, 4.70)
- moved J1 4.30 mm to (180.3, 17.1)
- moved R15 3.81 mm to (89.7, 19.9)
- moved R27 3.81 mm to (150.6, 19.9)
- moved R18 3.68 mm to (104.8, 19.9)
- moved R21 3.68 mm to (120.0, 19.9)
- moved R9 3.68 mm to (59.1, 19.9)
- moved R24 3.68 mm to (135.3, 19.9)
- moved R12 3.56 mm to (74.2, 19.9)
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- renumbered Q1 to Q9, Q2 to Q10, Q3 to Q11, Q4 to Q12, Q5 to Q13, Q6 to Q14, Q7 to Q15, Q8 to Q16
Connections:
- removed net +12V: IC1.1, J1.1, J3.1
- removed net SIG1: R4.1
- removed net SIG2: R7.1
- removed net SIG3: R10.1
- removed net SIG4: R13.1
- removed net SIG5: R16.1
- removed net SIG6: R19.1
- removed net SIG7: R22.1
- removed net SIG8: R25.1
- new net ARDUINO0: J4.3, U1.30
- new net ARDUINO1: U1.31
- new net ARDUINO14: R13.1, R31.2, U1.23
- new net ARDUINO15: R10.1, R30.2, U1.24
- new net ARDUINO16: R29.2, R7.1, U1.25
- new net ARDUINO17: R28.2, R4.1, U1.26
- new net ARDUINO18: J4.5, U1.27
- new net ARDUINO19: J4.4, U1.28
- new net ARDUINO3: J4.2, U1.1
- new net ARDUINO4: J4.1, U1.2
- new net ARDUINO5: R25.1, R35.2, U1.9
- new net ARDUINO6: R22.1, R34.2, U1.10
- new net ARDUINO7: J4.8, U1.11
- new net ARDUINO8: J4.7, U1.12
- new net ARDUINO9: J4.6, U1.13
- new net ARDUINOA6: R19.1, R33.2, U1.19
- new net ARDUINOA7: R16.1, R32.2, U1.22
- new net N$33: D1.A, R28.1
- new net N$34: D2.A, R29.1
- new net N$35: D3.A, R30.1
- new net N$36: D4.A, R31.1
- new net N$37: D5.A, R32.1
- new net N$38: D6.A, R33.1
- new net N$39: D7.A, R34.1
- new net N$40: D8.A, R35.1
- net +12VCC1: now also D10.C, D11.C, D12.C, D13.C, D14.C, D15.C, D16.C, D9.C, IC1.1, J1.1, J3.1, J5.3, J6.1, J6.2, J6.3, Q10.3, Q11.3, Q12.3, Q13.3, Q14.3, Q15.3, Q16.3, Q9.3; no longer Q10.2, Q11.2, Q12.2, Q13.2, Q14.2, Q15.2, Q16.2, Q9.2
- net GND: now also C5.1, D1.C, D2.C, D3.C, D4.C, D5.C, D6.C, D7.C, D8.C, J2.6, J5.2, J7.1, J7.2, J7.3; no longer J4.6
- net MISO: now also J2.1; no longer J4.1
- net MOSI: now also J2.4; no longer J4.4
- net N$11: now also D9.A
- net N$14: now also D10.A
- net N$17: now also D11.A
- net N$20: now also D12.A
- net N$23: now also D13.A
- net N$26: now also D14.A
- net N$29: now also D15.A
- net N$32: now also D16.A
- net OUTPUT1: now also Q9.2; no longer Q9.3
- net OUTPUT2: now also Q10.2; no longer Q10.3
- net OUTPUT3: now also Q11.2; no longer Q11.3
- net OUTPUT4: now also Q12.2; no longer Q12.3
- net OUTPUT5: now also Q13.2; no longer Q13.3
- net OUTPUT6: now also Q14.2; no longer Q14.3
- net OUTPUT7: now also Q15.2; no longer Q15.3
- net OUTPUT8: now also Q16.2; no longer Q16.3
- net RST: now also J2.5; no longer J4.5
- net SCK: now also J2.3; no longer J4.3
- net VCC: now also C5.2, J2.2, J5.1; no longer J4.2
Routing:
- net +12VCC1: track 0.00 -> 363.2 mm, vias 0 -> 13
- net CANL: track 0.00 -> 192.0 mm
- net CANH: track 0.00 -> 188.1 mm
- net GND: track 0.00 -> 128.4 mm, vias 0 -> 26
- net ARDUINO17: track 0.00 -> 94.1 mm, vias 0 -> 2
- net ARDUINO16: track 0.00 -> 76.9 mm, vias 0 -> 2
- net ARDUINO15: track 0.00 -> 53.4 mm
- net VCC: track 0.00 -> 52.7 mm, vias 0 -> 3
- net ARDUINO14: track 0.00 -> 37.9 mm
- net ARDUINO5: track 0.00 -> 28.8 mm
- net ARDUINO7: track 0.00 -> 25.3 mm, vias 0 -> 1
- net ARDUINO8: track 0.00 -> 24.6 mm, vias 0 -> 1
- net ARDUINO9: track 0.00 -> 24.1 mm, vias 0 -> 1
- net ARDUINO18: track 0.00 -> 22.7 mm, vias 0 -> 1
- net ARDUINOA7: track 0.00 -> 21.8 mm
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- added copper zone on layer 16, net GND
- added copper zone on layer 1, net VCC
Other:
- board size 196.8 x 40.3 mm -> 207 x 40.3 mm
- board text added: "1"
- board text added: "2"
- board text added: "3"
- board text added: "4"
