File: DigitalDash/ShifterControl.sch (EAGLE design)
At the start: 22 parts, among them IC1 7805T, J2 DT15-4P, J3 DT15-4P, J4 AVR_SPI_PROG_3X22X3_LOCK, U1 ATMEGA328P_TQFP, U2 MCP2515, U3 MCP2551, Y1 16MHz, Y2 8MHz

Commit message: add more cars
Parts:
- removed C3, C4: 22pF, SparkFun-Capacitors:22PF-0603-50V-5%
- removed J6: (no value), SparkFun-Connectors:CONN_063.5MM-6
- removed R1: 1k, SparkFun-Resistors:1KOHM-0603-1/10W-1%
- removed U1: ATMEGA328P_TQFP, SparkFun-IC-Microcontroller:ATMEGA328P_TQFP
- removed Y1: 16MHz, SparkFun-Clocks:CRYSTAL-8MHZSMD-HC49UP
- added C5: 470pF, SparkFun-Capacitors:22PF-0603-50V-5%
- added C7, C8: 22pF, SparkFun-Capacitors:22PF-0603-50V-5%
- added C9: 1uF, SparkFun-Capacitors:22PF-0603-50V-5%
- added R7: 1k, SparkFun-Resistors:1KOHM-0603-1/10W-1%
- added U4: ATMEGA328P_TQFP, SparkFun-IC-Microcontroller:ATMEGA328P_TQFP
- added X1, X2, X3: (no value), con-wago-500:W237-102
- added Y3: 16MHz, SparkFun-Clocks:CRYSTAL-8MHZSMD-HC49UP
Connections:
- removed net N$5: C4.2, U1.PB7(XTAL2/TOSC2), Y1.1
- removed net N$6: C3.2, U1.PB6(XTAL1/TOSC1), Y1.2
- new net N$10: C7.2, U4.PB6(XTAL1/TOSC1), Y3.2
- new net N$9: C8.2, U4.PB7(XTAL2/TOSC2), Y3.1
- net +12V: now also X2-1.KL; no longer J6.1
- net CAN_INT: now also U4.PD2(INT0); no longer U1.PD2(INT0)
- net CS: now also U4.PB2(SS/OC1B); no longer U1.PB2(SS/OC1B)
- net DATA: now also U4.PD5(T1); no longer U1.PD5(T1)
- net GND: now also C5.1, C7.1, C8.1, C9.1, U4.AGND, U4.AREF, U4.GND@3, U4.GND@5, X2-2.KL; no longer C3.1, C4.1, J6.2, U1.AGND, U1.AREF, U1.GND@3, U1.GND@5
- net LATCH: now also U4.PD6(AIN0); no longer U1.PD6(AIN0)
- net MCU_D: now also U4.PC0(ADC0); no longer U1.PC2(ADC2)
- net MCU_N: now also U4.PC1(ADC1); no longer U1.PC1(ADC1)
- net MCU_R: now also U4.PC2(ADC2); no longer U1.PC0(ADC0)
- net MISO: now also U4.PB4(MISO); no longer U1.PB4(MISO)
- net MOSI: now also U4.PB3(MOSI/OC2); no longer U1.PB3(MOSI/OC2)
- net RST: now also R7.2, U4.PC6(/RESET); no longer R1.2, U1.PC6(/RESET)
- net SCK: now also U4.PB5(SCK); no longer U1.PB5(SCK)
- net SHIFT_CLK: now also U4.PD7(AIN1); no longer U1.PD7(AIN1)
- net THROT_D: now also U$1.2-1, X1-2.KL; no longer J6.6, U$1.2-3
- net THROT_INPUT: now also X1-1.KL; no longer J6.3
- net THROT_N: now also X3-1.KL; no longer J6.5
- net THROT_R: now also U$1.2-3, X3-2.KL; no longer J6.4, U$1.2-1
- net VCC: now also C5.2, C9.2, R7.1, U4.AVCC, U4.VCC@4, U4.VCC@6; no longer R1.1, U1.AVCC, U1.VCC@4, U1.VCC@6
